File: board/OmniSCC+/OmniSCC+.kicad_pcb (KiCad board)
At the start: 2 copper layers, 99.8 x 46.4 mm, 28 parts, among them J1 Conn_MSX_BUS_edge, J2 Conn_01x20, J3 Conn_01x20, Q4 2N7002, U1 SN74LVC8T245, U2 SN74LVC8T245, U3 SN74LVC8T245, U4 SN74LVC8T245

Commit message: V2.0 update for OmniSCC and OmniSCC+
• Universal loaders with automatic MSX1 text / MSX2 graphical mode selection, refreshed UI and joystick support.
• Nextor support with direct access to the cartridge’s shared USB storage.
• Improved ROM compatibility: an external, updateable openMSX-based mapper database with custom entries, Generic 8 KB mapper support, and corrected Plain/48 KB ROM placement.
• KUC flash cartridge support with persistent .sav files, tested with Pampas & Selene variants.
• SCC-I/SCC+ support with 128 KB cartridge RAM and an independent fifth waveform.
• SCC volume adjustment using +/− in 10% steps, saved in the menu configuration.
• Improved DSK boot compatibility, configurable multi-disk switching with number keys, and independent drive B mounting with a diskette indicator.
• Polished loader rendering and Help, corrected filename truncation, and optional auto-start: delay=0 disables it.
• Unified O-prefixed BASIC/DOS disk commands and an updated example disk.
• Improved storage recovery, updated enclosures, and OmniSCC+ PCB revision 1.1 with a documented USB stability fix for revision 1.0.
Parts:
- added R7: 10K, Resistor_SMD:R_0805_2012Metric_Pad1.20x1.40mm_HandSolder, F.Cu at (86.5, 78.9)
Connections:
- J1 pad 11: /~{IORQ} -> unconnected-(J1-~{IORQ}-Pad11)
Routing:
- net /~{RES}: track 7.71 -> 44.0 mm, vias 1 -> 2
- net +5VA: track 190.8 -> 194.4 mm
Other:
- board text added: "2026-10 v1.1"
- board text removed: "2026-08 v1.0"
Changed lines of the file:
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@@
 	(title_block
 		(title "OmniSCC+")
-		(date "2026-08-31")
-		(rev "1.0")
+		(date "2026-10-15")
+		(rev "1.1")
 		(company "RBSC/OSPC.Club")
 	)
@@
 			(size 1.5 8)
 			(layers "B.Cu" "B.Mask")
-			(net "/~{IORQ}")
+			(net "unconnected-(J1-~{IORQ}-Pad11)")
 			(pinfunction "~{IORQ}_11")
-			(pintype "output")
+			(pintype "output+no_connect")
 		)
 		(pad "12" connect rect
@@
 		)
 	)
+	(footprint "Resistor_SMD:R_0805_2012Metric_Pad1.20x1.40mm_HandSolder"
+		(layer "F.Cu")
+		(at 86.525 78.875 -90)
+		(descr "Resistor SMD 0805 (2012 Metric), square (rectangular) end terminal, IPC-7351 nominal with elongated pad for handsoldering. (Body size source: IPC-SM-782 page 72, https://www.pcb-3d.com/wordpress/wp-content/uploads/ipc-sm-782a_amendment_1_and_2.pdf)")
+		(tags "resistor handsolder")
+		(property "Reference" "R7"
+			(at 0 -1.65 90)
+			(layer "F.SilkS")
+			(effects
+				(font
+					(size 1 1)
+					(thickness 0.15)
+				)
+			)
+		)
+		(property "Value" "10K"
+			(at 0 1.65 90)
+			(layer "F.Fab")
+			(effects
+				(font
+					(size 1 1)
+					(thickness 0.15)
+				)
+			)
+		)
+		(property "Datasheet" ""
+			(at 0 0 90)
+			(layer "F.Fab")
+			(hide yes)
+			(effects
+				(font
+					(size 1.27 1.27)
+				)
+			)
+		)
+		(property "Description" "Resistor"
+			(at 0 0 90)
+			(layer "F.Fab")
+			(hide yes)
+			(effects
+				(font
+					(size 1.27 1.27)
+				)
+			)
+		)
+		(property "KiLib_Generator" "SMD_2terminal_chip_molded"
+			(at 0 0 90)
+			(layer "F.SilkS")
+			(hide yes)
+			(effects
+				(font
+					(size 1 1)
+					(thickness 0.15)
+				)
+			)
+		)
+		(property ki_fp_filters "R_*")
+		(sheetname "/")
+		(sheetfile "OmniSCC+.kicad_sch")
+		(units
+			(unit
+				(name "A")
+				(pins "1" "2")
+			)
+		)
+		(attr smd)
+		(duplicate_pad_numbers_are_jumpers no)
+		(fp_line
+			(start -0.227064 0.735)
+			(end 0.227064 0.735)
+			(stroke
+				(width 0.12)
+				(type solid)
+			)
+			(layer "F.SilkS")
+		)
+		(fp_line
+			(start -0.227064 -0.735)
+			(end 0.227064 -0.735)
+			(stroke
+				(width 0.12)
+				(type solid)
+			)
+			(layer "F.SilkS")
+		)
+		(fp_rect
+			(start -1.85 -0.95)
+			(end 1.85 0.95)
+			(stroke
+				(width 0.05)
+				(type solid)
+			)
+			(fill no)
+			(layer "F.CrtYd")
+		)
+		(fp_rect
+			(start -1 -0.625)
+			(end 1 0.625)
+			(stroke
+				(width 0.1)
+				(type solid)
+			)
+			(fill no)
+			(layer "F.Fab")
+		)
+		(fp_text user "${REFERENCE}"
+			(at 0 0 90)
+			(layer "F.Fab")
+			(effects
+				(font
+					(size 0.5 0.5)
+					(thickness 0.08)
+				)
+			)
+		)
+		(pad "1" smd roundrect
+			(at -1 0 270)
+			(size 1.2 1.4)
+			(layers "F.Cu" "F.Mask" "F.Paste")
+			(roundrect_rratio 0.208333)
+			(net "+5VA")
+			(pintype "passive")
+		)
+		(pad "2" smd roundrect
+			(at 1 0 270)
+			(size 1.2 1.4)
+			(layers "F.Cu" "F.Mask" "F.Paste")
+			(roundrect_rratio 0.208333)
+			(net "/~{RES}")
+			(pintype "passive")
+		)
+		(embedded_fonts no)
+		(model "${KICAD10_3DMODEL_DIR}/Resistor_SMD.3dshapes/R_0805_2012Metric.step"
+			(offset
+				(xyz 0 0 0)
+			)
+			(scale
+				(xyz 1 1 1)
+			)
+			(rotate
+				(xyz 0 0 0)
+			)
+		)
+	)
 	(footprint "Capacitor_SMD:C_0805_2012Metric"
 		(layer "F.Cu")
@@
 		)
 	)
-	(gr_text "2026-08 v1.0"
+	(gr_text "2026-10 v1.1"
 		(at 54.5 63 0)
 		(layer "F.SilkS")
@@
 	(segment
 		(start 81.45 78.35)
-		(end 86.5 73.3)
+		(end 84.9 74.9)
 		(width 1)
 		(layer "F.Cu")
@@
 	)
 	(segment
+		(start 84.9 74.9)
+		(end 86.525 76.525)
+		(width 1)
+		(layer "F.Cu")
+		(net "+5VA")
+	)
+	(segment
 		(start 86.5 73.3)
 		(end 86.5 72.5)
@@
 	)
 	(segment
+		(start 86.525 76.525)
+		(end 86.525 77.875)
+		(width 1)
+		(layer "F.Cu")
+		(net "+5VA")
+	)
+	(segment
 		(start 126.425 79.824)
 		(end 126.5 79.749)
@@
 	)
 	(segment
+		(start 84.9 74.9)
+		(end 86.5 73.3)
+		(width 1)
+		(layer "F.Cu")
+		(net "+5VA")
+	)
+	(segment
 		(start 104.5 79.5)
 		(end 105 79.5)
@@
 	)
 	(segment
+		(start 87.875 79.875)
+		(end 86.525 79.875)
+		(width 0.25)
+		(layer "F.Cu")
+		(net "/~{RES}")
+	)
+	(segment
+		(start 89 81)
+		(end 87.875 79.875)
+		(width 0.25)
+		(layer "F.Cu")
+		(net "/~{RES}")
+	)
+	(segment
 		(start 121.5 83)
 		(end 121.875 82.625)
@@
 		(net "/~{RES}")
 	)
+	(via
+		(at 89 81)
+		(size 0.8)
+		(drill 0.4)
+		(layers "F.Cu" "B.Cu")
+		(net "/~{RES}")
+	)
 	(segment
 		(start 120.98 83.52)
@@
 	)
 	(segment
+		(start 121.5 83)
+		(end 119.5 81)
+		(width 0.25)
+		(layer "B.Cu")
+		(net "/~{RES}")
+	)
+	(segment
 		(start 120.98 88.2)
 		(end 120.98 83.52)
 		(width 0.25)
 		(layer "B.Cu")
+		(net "/~{RES}")
+	)
+	(segment
+		(start 119.5 81)
+		(end 89 81)
+		(width 0.25)
+		(layer "B.Cu")
