File: board/OmniSCC+/OmniSCC+.kicad_sch (KiCad schematic)
At the start: 28 parts, among them J1 Conn_MSX_BUS_edge, J2 Conn_01x20, J3 Conn_01x20, Q4 2N7002, U1 SN74LVC8T245, U2 SN74LVC8T245, U3 SN74LVC8T245, U4 SN74LVC8T245

Commit message: V2.0 update for OmniSCC and OmniSCC+
• Universal loaders with automatic MSX1 text / MSX2 graphical mode selection, refreshed UI and joystick support.
• Nextor support with direct access to the cartridge’s shared USB storage.
• Improved ROM compatibility: an external, updateable openMSX-based mapper database with custom entries, Generic 8 KB mapper support, and corrected Plain/48 KB ROM placement.
• KUC flash cartridge support with persistent .sav files, tested with Pampas & Selene variants.
• SCC-I/SCC+ support with 128 KB cartridge RAM and an independent fifth waveform.
• SCC volume adjustment using +/− in 10% steps, saved in the menu configuration.
• Improved DSK boot compatibility, configurable multi-disk switching with number keys, and independent drive B mounting with a diskette indicator.
• Polished loader rendering and Help, corrected filename truncation, and optional auto-start: delay=0 disables it.
• Unified O-prefixed BASIC/DOS disk commands and an updated example disk.
• Improved storage recovery, updated enclosures, and OmniSCC+ PCB revision 1.1 with a documented USB stability fix for revision 1.0.
Parts:
- added R7: 10K, Resistor_SMD:R_0805_2012Metric_Pad1.20x1.40mm_HandSolder, symbol Device:R
Connections:
- net +5VA: now also R7.1
- net ~{RES}: now also R7.2
Changed lines of the file:
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@@
 		(title "OmniSCC+")
 		(date "2026-08-31")
-		(rev "1.0")
+		(rev "1.1")
 	)
 	(text "<---"
@@
 	)
 	(junction
+		(at 36.83 58.42)
+		(diameter 0)
+		(color 0 0 0 0)
+	)
+	(junction
 		(at 67.31 172.72)
 		(diameter 0)
@@
 	(wire
 		(pts
+			(xy 36.83 45.72) (xy 36.83 48.26)
+		)
+		(stroke
+			(width 0)
+			(type default)
+		)
+	)
+	(wire
+		(pts
 			(xy 86.36 73.66) (xy 93.98 73.66)
 		)
@@
 	(wire
 		(pts
+			(xy 36.83 58.42) (xy 55.88 58.42)
+		)
+		(stroke
+			(width 0)
+			(type default)
+		)
+	)
+	(wire
+		(pts
 			(xy 213.36 100.33) (xy 210.82 100.33)
 		)
@@
 	(wire
 		(pts
+			(xy 36.83 55.88) (xy 36.83 58.42)
+		)
+		(stroke
+			(width 0)
+			(type default)
+		)
+	)
+	(wire
+		(pts
 			(xy 55.88 148.59) (xy 67.31 148.59)
 		)
@@
 	(wire
 		(pts
-			(xy 48.26 58.42) (xy 55.88 58.42)
+			(xy 26.67 58.42) (xy 36.83 58.42)
 		)
 		(stroke
@@
 	)
 	(label "~{RES}"
-		(at 48.26 58.42 0)
+		(at 26.67 58.42 0)
 		(effects
 			(font
@@
 	)
 	(symbol
+		(lib_id "power:+5VA")
+		(at 36.83 45.72 0)
+		(unit 1)
+		(body_style 1)
+		(exclude_from_sim no)
+		(in_bom yes)
+		(on_board yes)
+		(in_pos_files yes)
+		(dnp no)
+		(fields_autoplaced yes)
+		(property "Reference" "#PWR036"
+			(at 36.83 49.53 0)
+			(hide yes)
+			(show_name no)
+			(do_not_autoplace no)
+			(effects
+				(font
+					(size 1.27 1.27)
+				)
+			)
+		)
+		(property "Value" "+5VA"
+			(at 36.83 40.64 0)
+			(show_name no)
+			(do_not_autoplace no)
+			(effects
+				(font
+					(size 1.27 1.27)
+				)
+			)
+		)
+		(property "Footprint" ""
+			(at 36.83 45.72 0)
+			(hide yes)
+			(show_name no)
+			(do_not_autoplace no)
+			(effects
+				(font
+					(size 1.27 1.27)
+				)
+			)
+		)
+		(property "Datasheet" ""
+			(at 36.83 45.72 0)
+			(hide yes)
+			(show_name no)
+			(do_not_autoplace no)
+			(effects
+				(font
+					(size 1.27 1.27)
+				)
+			)
+		)
+		(property "Description" "Power symbol creates a global label with name \"+5VA\""
+			(at 36.83 45.72 0)
+			(hide yes)
+			(show_name no)
+			(do_not_autoplace no)
+			(effects
+				(font
+					(size 1.27 1.27)
+				)
+			)
+		)
+		(pin "1"
+		)
+		(instances
+			(project "OmniSCC+"
+				(path "/6ab751e5-e6a2-456a-a8ab-7e7d5e1fa70a"
+					(reference "#PWR036")
+					(unit 1)
+				)
+			)
+		)
+	)
+	(symbol
 		(lib_id "power:GND")
 		(at 248.92 83.82 0)
@@
 					(unit 1)
 				)
+			)
+		)
+	)
+	(symbol
+		(lib_id "Device:R")
+		(at 36.83 52.07 0)
+		(unit 1)
+		(body_style 1)
+		(exclude_from_sim no)
+		(in_bom yes)
+		(on_board yes)
+		(in_pos_files yes)
+		(dnp no)
+		(fields_autoplaced yes)
+		(property "Reference" "R7"
+			(at 39.37 50.7999 0)
+			(show_name no)
+			(do_not_autoplace no)
+			(effects
+				(font
+					(size 1.27 1.27)
+				)
+				(justify left)
+			)
+		)
+		(property "Value" "10K"
+			(at 39.37 53.3399 0)
+			(show_name no)
+			(do_not_autoplace no)
+			(effects
+				(font
+					(size 1.27 1.27)
+				)
+				(justify left)
+			)
+		)
+		(property "Footprint" "Resistor_SMD:R_0805_2012Metric_Pad1.20x1.40mm_HandSolder"
+			(at 35.052 52.07 90)
+			(hide yes)
+			(show_name no)
+			(do_not_autoplace no)
+			(effects
+				(font
+					(size 1.27 1.27)
+				)
+			)
+		)
+		(property "Datasheet" ""
+			(at 36.83 52.07 0)
+			(hide yes)
+			(show_name no)
+			(do_not_autoplace no)
+			(effects
+				(font
+					(size 1.27 1.27)
+				)
+			)
+		)
+		(property "Description" "Resistor"
+			(at 36.83 52.07 0)
+			(hide yes)
+			(show_name no)
+			(do_not_autoplace no)
+			(effects
+				(font
+					(size 1.27 1.27)
+				)
+			)
+		)
+		(pin "2"
+		)
+		(pin "1"
+		)
+		(instances
+			(project "OmniSCC+"
+				(path "/6ab751e5-e6a2-456a-a8ab-7e7d5e1fa70a"
+					(reference "R7")
+					(unit 1)
+				)
